File: PCB/SaponseEx.kicad_sch (KiCad schematic)
At the start: 52 parts, among them J1 CONN_BATT, J2 Conn_A_Main, J3 Conn_B_Main, M1 Fan, M2 MK06-4.5, M3 MK06-4.5, Q1 BSS138, Q2 BSS138, Q3 BSS138, Q4 BSS138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

Commit message: [fix]壁センサの配線ミスを修正
Connections:
- net +3V3: now also U1.4, U2.4, U3.4, U4.4; no longer U1.3, U2.3, U3.3, U4.3
- net GND: now also U6.3; no longer U6.2
- net SENS_FL: now also U2.3; no longer U2.4
- net SENS_FR: now also U3.3; no longer U3.4
- net SENS_L: now also U1.3; no longer U1.4
- net SENS_R: now also U4.3; no longer U4.4
- net at Q5.1 (G), R3.2: now also U6.2; no longer U6.3

Commit message: [fix]壁制御のゲインを調整
Parts:
- R11, R13, R7, R9: value 1M -> 1k
- R5: value 10k -> 20k
Changed lines of the file:
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@@
       (effects (font (size 1.27 1.27)) (justify left))
     )
-    (property "Value" "1M" (id 1) (at 62.23 57.15 90))
+    (property "Value" "1k" (id 1) (at 62.23 57.15 90))
     (property "Footprint" "Resistor_SMD:R_0603_1608Metric_Pad0.98x0.95mm_HandSolder" (id 2) (at 60.452 57.15 90)
       (effects (font (size 1.27 1.27)) hide)
@@
       (effects (font (size 1.27 1.27)) (justify left))
     )
-    (property "Value" "1M" (id 1) (at 157.48 57.15 90))
+    (property "Value" "1k" (id 1) (at 157.48 57.15 90))
     (property "Footprint" "Resistor_SMD:R_0603_1608Metric_Pad0.98x0.95mm_HandSolder" (id 2) (at 155.702 57.15 90)
       (effects (font (size 1.27 1.27)) hide)
@@
       (effects (font (size 1.27 1.27)) (justify left))
     )
-    (property "Value" "1M" (id 1) (at 93.98 57.15 90))
+    (property "Value" "1k" (id 1) (at 93.98 57.15 90))
     (property "Footprint" "Resistor_SMD:R_0603_1608Metric_Pad0.98x0.95mm_HandSolder" (id 2) (at 92.202 57.15 90)
       (effects (font (size 1.27 1.27)) hide)
@@
       (effects (font (size 1.27 1.27)) (justify left))
     )
-    (property "Value" "1M" (id 1) (at 125.73 57.15 90))
+    (property "Value" "1k" (id 1) (at 125.73 57.15 90))
     (property "Footprint" "Resistor_SMD:R_0603_1608Metric_Pad0.98x0.95mm_HandSolder" (id 2) (at 123.952 57.15 90)
       (effects (font (size 1.27 1.27)) hide)
@@
       (effects (font (size 1.27 1.27)) (justify left))
     )
-    (property "Value" "10k" (id 1) (at 208.28 48.26 90))
+    (property "Value" "20k" (id 1) (at 208.28 48.26 90))
     (property "Footprint" "Resistor_SMD:R_0603_1608Metric_Pad0.98x0.95mm_HandSolder" (id 2) (at 206.502 48.26 90)
       (effects (font (size 1.27 1.27)) hide)
@@
     )
     (path "/77320cbf-7898-4a50-9ca9-25795e54086e"
-      (reference "R5") (unit 1) (value "10k") (footprint "Resistor_SMD:R_0603_1608Metric_Pad0.98x0.95mm_HandSolder")
+      (reference "R5") (unit 1) (value "20k") (footprint "Resistor_SMD:R_0603_1608Metric_Pad0.98x0.95mm_HandSolder")
     )
     (path "/56768922-193f-42d1-a7ea-fd3dea8fa472"
@@
     )
     (path "/0024a0f9-0ae2-4852-bd64-407eaebf17fc"
-      (reference "R7") (unit 1) (value "1M") (footprint "Resistor_SMD:R_0603_1608Metric_Pad0.98x0.95mm_HandSolder")
+      (reference "R7") (unit 1) (value "1k") (footprint "Resistor_SMD:R_0603_1608Metric_Pad0.98x0.95mm_HandSolder")
     )
     (path "/c40708ea-f8d2-464e-8670-0ea16844230f"
@@
     )
     (path "/0d0553d5-6133-4c5d-8c2a-6490ec839c9d"
-      (reference "R9") (unit 1) (value "1M") (footprint "Resistor_SMD:R_0603_1608Metric_Pad0.98x0.95mm_HandSolder")
+      (reference "R9") (unit 1) (value "1k") (footprint "Resistor_SMD:R_0603_1608Metric_Pad0.98x0.95mm_HandSolder")
     )
     (path "/e1087e7f-b87f-4202-ac2d-e5282f5c459b"
@@
     )
     (path "/660936b5-1053-410e-b89e-85604a61cc29"
-      (reference "R11") (unit 1) (value "1M") (footprint "Resistor_SMD:R_0603_1608Metric_Pad0.98x0.95mm_HandSolder")
+      (reference "R11") (unit 1) (value "1k") (footprint "Resistor_SMD:R_0603_1608Metric_Pad0.98x0.95mm_HandSolder")
     )
     (path "/e6a1bb02-f2fe-4aa8-8c5f-c7ed41f9d733"
@@
     )
     (path "/0c211606-aecf-4041-b3a9-495dc757bd62"
-      (reference "R13") (unit 1) (value "1M") (footprint "Resistor_SMD:R_0603_1608Metric_Pad0.98x0.95mm_HandSolder")
+      (reference "R13") (unit 1) (value "1k") (footprint "Resistor_SMD:R_0603_1608Metric_Pad0.98x0.95mm_HandSolder")
     )
     (path "/89f6357d-b99b-404c-b50c-558bfc4b555d"
